File: Nibbler-3.3V.sch (KiCad schematic (older format))
At the start: 11 parts, among them J1 CONN_01X04, J2 +3.3, J3 GND, Q1 UM6K33N, Q2 UM6K33N

Commit message: Minor layout rework - rotated current limit resistor in layout and reversed LED connections in schematic. Modified bottom silkscreen text
Parts:
- D1, D2, D3, D4: Part # LG R971-KN-1 -> (none); Part Number (none) -> LG R971-KN-1
- J1: Part Number (none) -> PRPC004SBAN-M71RC
- Q1, Q2: Part Number (none) -> UM6K33NTN
- RN1: Part # YC164-JR-0775RL -> (none); Part Number (none) -> YC164-JR-0775RL
- RN2: Part # YC164-JR-0710KL -> (none); Part Number (none) -> YC164-JR-0710KL
Other:
- note added: "Design Parameters:\nLED Vf (V) If (mA) PN\nGreen 2.2 14.6 LG R971-KN-1\nRed 2.0 17.3 LS R976-NR-1"
- moved on the sheet: D1, D2, D3, D4, J1, J2, J3, Q1, Q2, RN1, RN2
